File: hoop.brd (EAGLE design)
At the start: 56 x 56 mm, 33 parts, among them U1 PIC32MM0064GPL020-I/ML, U2 SGM2200

Commit message: Cleaning up pcb files
Parts:
- removed R10, R11, R12, R4, R5, R6, R7, R8, R9: (no value), rcl:R0805
- removed R13: (no value), rcl:R0402
- added C10, C4, C5, C6, C7, C8, C9: (no value), rcl:C0805
- added D13, D14, D15, D16, D17, D18, D19, D20, D21, D22, D23, D24, D25, D26, D27, D28, D29, D30, D31, D32, D33, D34, D35, D36, D37, D38, D39, D40, D41, D42, D43, D44, D45, D46, D47, D48, D49, D50, D51, D52, D53, D54, D55, D56, D57, D58, D59, D60: SMD-LX0707RGB-TR, earring:SMD-LX0707RGB-TR
- added J1: JMP, earring:SOLDER_JMP
- added L1: (no value), rcl:L3216C
- added U3: ATTINY202, earring:SOIC127P600X175-8N
- C1, C2, C3: device rcl:C0402 -> rcl:C0805
- D1, D10, D11, D12, D2, D3, D4, D5, D6, D7, D8, D9: value FM-Z2727RGBA-SH -> SMD-LX0707RGB-TR; device earring:SMD_2.8X2.7MM -> earring:SMD-LX0707RGB-TR
- U1: value PIC32MM0064GPL020-I/ML -> LTC3525; device earring:QFN50P400X400X100-21T280N -> earring:SOP65P210X100-6N
- U2: value SGM2200 -> MXC6255XU; device earring:SOT23 -> earring:RESCAV110P300X300X105-6N
- moved U2 42.4 mm to (46.9, 38.9), turned to 240 degrees
- moved D12 40.9 mm to (6.62, 25.8), turned to 276 degrees
- moved D1 37.2 mm to (17.2, 46.6), turned to 210 degrees
- moved D11 37.2 mm to (6.50, 28.0), turned to 270 degrees
- moved C3 35.2 mm to (9.21, 39.0), turned to 205 degrees
- moved U1 34.5 mm to (6.65, 36.1), turned to 110 degrees
- moved C1 32.9 mm to (6.41, 29.5), turned to 185 degrees
- moved D2 32.0 mm to (15.4, 45.4), turned to 216 degrees
- moved D10 32.0 mm to (6.62, 30.2), turned to 264 degrees
- moved R1 28.3 mm to (25.8, 50.1), flipped to the bottom, turned to 180 degrees
- moved C2 27.9 mm to (6.75, 31.8), turned to 190 degrees
- moved D3 25.3 mm to (13.6, 44.0), turned to 222 degrees
- moved D9 25.3 mm to (6.97, 32.5), turned to 258 degrees
- moved D8 17.5 mm to (7.55, 34.6), turned to 252 degrees
- moved D4 17.5 mm to (12.0, 42.4), turned to 228 degrees
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Connections:
- removed net +3V3: C1.1, R13.2, U1.17, U2.2
- removed net /MCLR: C2.1, R13.1, U1.18
- removed net G1P1: D2.G+, D3.G+, D4.R+, R1.2, U1.14
- removed net G1P2: D1.G+, D3.B+, D4.G+, R2.2, U1.8
- removed net G1P3: D1.B+, D2.B+, D4.B+, R3.2, U1.3
- removed net G1P4: D1.R+, D2.R+, D3.R+, R4.2, U1.15
- removed net G2P1: D6.R+, D7.R+, D8.R+, R5.2, U1.20
- removed net G2P2: D5.R+, D7.G+, D8.G+, R6.2, U1.1
- removed net G2P3: D5.G+, D6.G+, D8.B+, R7.2, U1.19
- removed net G2P4: D5.B+, D6.B+, D7.B+, R8.2, U1.2
- removed net G3P1: D10.R+, D11.R+, D12.G+, R9.2, U1.12
- removed net G3P2: D11.G+, D12.R+, D9.R+, R10.2, U1.13
- removed net G3P3: D10.G+, D12.B+, D9.G+, R11.2, U1.10
- removed net G3P4: D10.B+, D11.B+, D9.B+, R12.2, U1.9
- removed net N$27: B3.POS1, B3.POS2, U2.3
- removed net PGEC: U1.7
- removed net PGED: U1.6
- new net LED_DATA: D1.3, U3.3
- new net N$13: D15.1, D16.3
- new net N$14: D16.1, D17.3
- new net N$15: D17.1, D18.3
- new net N$16: D19.1, D20.3
- new net N$20: D23.1, D24.3
- new net N$21: D25.1, D26.3
- new net N$22: D26.1, D27.3
- new net N$23: D27.1, D28.3
- new net N$24: D28.1, D29.3
- new net N$28: D29.1, D30.3
- new net N$29: D31.1, D32.3
- new net N$30: D32.1, D33.3
- new net N$31: D33.1, D34.3
- new net N$32: D34.1, D35.3
- new net N$33: D35.1, D36.3
- new net N$34: D37.1, D38.3
- new net N$35: D38.1, D39.3
- new net N$36: D39.1, D40.3
- new net N$37: D40.1, D41.3
- new net N$38: D41.1, D42.3
- new net N$39: D43.1, D44.3
- new net N$40: D44.1, D45.3
- new net N$41: D45.1, D46.3
- new net N$42: D46.1, D47.3
- new net N$43: D47.1, D48.3
- new net N$44: D49.1, D50.3
- new net N$45: D50.1, D51.3
- new net N$46: D51.1, D52.3
- new net N$47: D52.1, D53.3
- new net N$48: D53.1, D54.3
- new net N$49: D55.1, D56.3
- new net N$5: D5.1, D6.3
- new net N$50: D56.1, D57.3
- new net N$51: D57.1, D58.3
- new net N$52: D58.1, D59.3
- new net N$53: D59.1, D60.3
- new net N$54: D6.1, D7.3
- new net N$55: D12.1, D13.3
- new net N$56: D18.1, D19.3
- new net N$57: D24.1, D25.3
- new net N$58: D30.1, D31.3
- new net N$59: D36.1, D37.3
- new net N$60: D42.1, D43.3
- new net N$61: D48.1, D49.3
- new net N$62: D54.1, D55.3
- new net N$64: L1.2, U1.6
- new net N$66: U2.1, U3.7
- new net N$69: R1.1, U3.6
- new net N$8: D10.3, D9.1
- new net SCL: R3.1, U2.4, U3.5
- new net SDA: R2.1, U2.5, U3.4
- new net UPDI: J1.P$2, R1.2
- new net VBAT: B3.POS1, B3.POS2, C1.1, C2.1, L1.1, U1.1, U1.3
- new net VCC: C10.1, C3.1, C4.1, C5.1, C6.1, C7.1, C8.1, C9.1, D1.2, D10.2, D11.2, D12.2, D13.2, D14.2, D15.2, D16.2, D17.2, D18.2, D19.2, D2.2, D20.2, D21.2, D22.2, D23.2, D24.2, D25.2, D26.2, D27.2, D28.2, D29.2, D3.2, D30.2, D31.2, D32.2, D33.2, D34.2, D35.2, D36.2, D37.2, D38.2, D39.2, D4.2, D40.2, D41.2, D42.2, D43.2, D44.2, D45.2, D46.2, D47.2, D48.2, D49.2, D5.2, D50.2, D51.2, D52.2, D53.2, D54.2, D55.2, D56.2, D57.2, D58.2, D59.2, D6.2, D60.2, D7.2, D8.2, D9.2, J1.P$1, R2.2, R3.2, U1.4, U2.3, U3.1
- net GND: now also C10.2, C3.2, C4.2, C5.2, C6.2, C7.2, C8.2, C9.2, D1.4, D10.4, D11.4, D12.4, D13.4, D14.4, D15.4, D16.4, D17.4, D18.4, D19.4, D2.4, D20.4, D21.4, D22.4, D23.4, D24.4, D25.4, D26.4, D27.4, D28.4, D29.4, D3.4, D30.4, D31.4, D32.4, D33.4, D34.4, D35.4, D36.4, D37.4, D38.4, D39.4, D4.4, D40.4, D41.4, D42.4, D43.4, D44.4, D45.4, D46.4, D47.4, D48.4, D49.4, D5.4, D50.4, D51.4, D52.4, D53.4, D54.4, D55.4, D56.4, D57.4, D58.4, D59.4, D6.4, D60.4, D7.4, D8.4, D9.4, U1.2, U1.5, U2.6, U3.8; no longer C3.1, U1.16, U2.1
- net N$1: now also D1.1, D2.3; no longer D1.B-, D1.G-, D1.R-, R1.1
- net N$10: now also D11.1, D12.3; no longer D6.B-, D6.G-, D6.R-, R6.1
- net N$11: now also D13.1, D14.3; no longer D7.B-, D7.G-, D7.R-, R7.1
- net N$12: now also D14.1, D15.3; no longer D8.B-, D8.G-, D8.R-, R8.1
- net N$17: now also D20.1, D21.3; no longer D9.B-, D9.G-, D9.R-, R9.1
- net N$18: now also D21.1, D22.3; no longer D10.B-, D10.G-, D10.R-, R10.1
- net N$19: now also D22.1, D23.3; no longer D11.B-, D11.G-, D11.R-, R11.1
- net N$2: now also D2.1, D3.3; no longer C3.2, U1.11
- net N$3: now also D3.1, D4.3; no longer D2.B-, D2.G-, D2.R-, R2.1
- net N$4: now also D4.1, D5.3; no longer D4.B-, D4.G-, D4.R-, R4.1
- net N$6: now also D7.1, D8.3; no longer D3.B-, D3.G-, D3.R-, R3.1
- net N$7: now also D8.1, D9.3; no longer D12.B-, D12.G-, D12.R-, R12.1
- net N$9: now also D10.1, D11.3; no longer D5.B-, D5.G-, D5.R-, R5.1
Routing:
- net VCC: track 0.00 -> 235.7 mm, vias 0 -> 11
- net GND: track 17.1 -> 201.6 mm, vias 3 -> 26
- net G3P4: track 82.8 -> 0.00 mm, vias 5 -> 0
- net G3P3: track 77.7 -> 0.00 mm, vias 1 -> 0
- net G2P4: track 72.2 -> 0.00 mm, vias 1 -> 0
- net G3P1: track 69.8 -> 0.00 mm, vias 3 -> 0
- net G3P2: track 68.3 -> 0.00 mm, vias 1 -> 0
- net G2P2: track 60.5 -> 0.00 mm, vias 3 -> 0
- net G2P3: track 59.1 -> 0.00 mm, vias 2 -> 0
- net G1P3: track 58.9 -> 0.00 mm, vias 1 -> 0
- net G2P1: track 55.9 -> 0.00 mm, vias 1 -> 0
- net G1P2: track 47.5 -> 0.00 mm, vias 1 -> 0
- net G1P4: track 44.6 -> 0.00 mm, vias 1 -> 0
- net +3V3: track 42.5 -> 0.00 mm, vias 1 -> 0
- net SDA: track 0.00 -> 38.8 mm
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- added copper zone on layer 1, net N$69
- added copper zone on layer 1, net PAD
- added copper zone on layer 1, net UPDI
- added copper zone on layer 1, net VBAT
- added copper zone on layer 16, net VBAT
- added copper zone on layer 1, net VCC
- added copper zone on layer 16, net VCC
- removed copper zone on layer 1, net +3V3
- removed copper zone on layer 1, net /MCLR
- removed copper zone on layer 16, net N$27
- removed copper zone on layer 1, net PAD0
- removed copper zone on layer 1, net PAD3
- removed copper zone on layer 1, net PGEC
- removed copper zone on layer 1, net PGED
Other:
- board text added: "to m who lights up my life <3 b 4.8.21"
- board text removed: "To Mandie, who lights up my life -B"
